File: OpenThermalCamera.kicad_pcb (KiCad board)
At the start: 2 copper layers, 26 x 20 mm, 23 parts, among them J1 Conn_ARM_JTAG_SWD_10, J2 DX07P024AJ1R1500, SW1 PB_Bootloader, U1 MLX90640, U2 TPS793333-EP, U3 STM32F042F6Px, U4 NUP2202

Commit message: Preperations for Rev3
Other:
- rule pad_to_mask_clearance: 0.2 -> 0.05
Changed lines of the file:
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@@
     (pad_size 1.2 1.2)
     (pad_drill 0.7)
-    (pad_to_mask_clearance 0.2)
+    (pad_to_mask_clearance 0.05)
     (aux_axis_origin 0 0)
     (visible_elements 7FFFFFFF)

Commit message: First Rev3-M commit
Parts:
- removed R4: 5k1, Resistor_SMD:R_0805_2012Metric_Pad1.15x1.40mm_HandSolder
- G1: value (none) -> Logo_Open_Hardware_Small
- J2: value DX07P024AJ1R1500 -> reversible_micro_usb; footprint lib_fp:DX07P024AJ1R1500 -> lib_fp:reversible_micro_usb
- moved J2 2.91 mm to (40.0, 26.6), turned to 0 degrees
Connections:
- J2 pad A1: GND -> +5V
- J2 pad A2: Net-(J2-PadA2) -> /USB_N
- J2 pad A3: Net-(J2-PadA3) -> /USB_P
- J2 pad A4: +5V -> GND
- J2 pad A5: Net-(J2-PadA5) -> GND
- J2 pad B1: GND -> +5V
- J2 pad B2: Net-(J2-PadB2) -> /USB_N
- J2 pad B3: Net-(J2-PadB3) -> /USB_P
- J2 pad B4: +5V -> GND
- J2 pad B5: Net-(J2-PadB5) -> GND
- U4 pad 1: /USB_P -> /USB_N
- U4 pad 6: /USB_N -> /USB_P
Routing:
- net Net-(J2-PadA5): track 10.3 -> 0.00 mm, vias 1 -> 0
- net GND: track 82.0 -> 74.0 mm, vias 12 -> 14
- net +5V: track 46.0 -> 39.1 mm
- net /USB_N: track 27.9 -> 33.0 mm, vias 1 -> 2
- net /USB_P: track 26.5 -> 29.6 mm, vias 1 -> 2
Other:
- board size 26 x 20 mm -> 26 x 21.5 mm
- board text added: "OTC Rev3-M"
- board text removed: "OTC Rev3"
