File: OpenThermalCamera.sch (KiCad schematic (older format))
At the start: 18 parts, among them J1 Conn_ARM_JTAG_SWD_10, J2 USB_CONN, SW1 PB_Bootloader, U1 MLX90640, U2 TPS793333-EP, U3 STM32F042F6Px, U4 NUP2202

Commit message: Rev2
Parts:
- removed J2: USB_CONN, usb_b2b_connector:usb_b2b_connector, symbol Connector_Generic:Conn_01x04
- added D1: LED_Dual_ACAC, LED_SMD:LED_Cree-PLCC4_2x2mm_CW, symbol Device:LED_Dual_ACAC
- added G1: Logo_Open_Hardware_Small, Symbol:OSHW-Logo2_7.3x6mm_SilkScreen, symbol Graphic:Logo_Open_Hardware_Small
- added J2: DX07P024AJ1R1500, lib_fp:DX07P024AJ1R1500, symbol DX07P024AJ1R1500:DX07P024AJ1R1500
- added R4: 5k1, Resistor_SMD:R_0805_2012Metric_Pad1.15x1.40mm_HandSolder, symbol Device:R
- added R5: 10R, Resistor_SMD:R_0805_2012Metric_Pad1.15x1.40mm_HandSolder, symbol Device:R
- added R6: 130R, Resistor_SMD:R_0805_2012Metric_Pad1.15x1.40mm_HandSolder, symbol Device:R
- SW1: footprint Button_Switch_SMD:SW_SPST_FSMSM -> Jumper:SolderJumper-2_P1.3mm_Open_RoundedPad1.0x1.5mm
- U1: footprint Package_TO_SOT_THT:TO-39-4_Window -> lib_fp:MLX90640; symbol mlx90640:MLX90640 -> MLX90640:MLX90640
Connections:
- net labels added: BLUE_LED, RED_LED
- wire segments 47 -> 58
- no-connect marks 3 -> 22
Other:
- note added: "Indicator Blue/Red LED"
- moved on the sheet: C1, C2, C3, C4, C5, C6, MH1, MH2, R1, R2, R3, SW1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

Commit message: First Rev3-M commit
Parts:
- removed J2: DX07P024AJ1R1500, lib_fp:DX07P024AJ1R1500, symbol DX07P024AJ1R1500:DX07P024AJ1R1500
- removed R4: 5k1, Resistor_SMD:R_0805_2012Metric_Pad1.15x1.40mm_HandSolder, symbol Device:R
- added J2: reversible_micro_usb, lib_fp:reversible_micro_usb, symbol reversible_micro_usb:reversible_micro_usb
Connections:
- wire segments 58 -> 70
- no-connect marks 22 -> 11
Other:
- moved on the sheet: U4
Changed lines of the file:
@@
 	3150 3200 3050 3200
-$Comp
-L power:+5V #PWR0112
-U 1 1 5B955DC4
-P 13750 6300
-F 0 "#PWR0112" H 13750 6150 50  0001 C CNN
-F 1 "+5V" H 13765 6473 50  0000 C CNN
-F 2 "" H 13750 6300 50  0001 C CNN
-F 3 "" H 13750 6300 50  0001 C CNN
-	1    13750 6300
-	1    0    0    -1
-$EndComp
-Text Label 12400 7150 2    50   ~ 0
-USB_N
-Text Label 12400 7250 2    50   ~ 0
-USB_P
-$Comp
-L power:GND #PWR0113
-U 1 1 5B9575B1
-P 13750 7750
-F 0 "#PWR0113" H 13750 7500 50  0001 C CNN
-F 1 "GND" H 13755 7577 50  0000 C CNN
-F 2 "" H 13750 7750 50  0001 C CNN
-F 3 "" H 13750 7750 50  0001 C CNN
-	1    13750 7750
-	1    0    0    -1
-$EndComp
 $Comp
 L Power_Protection:NUP2202 U4
 U 1 1 5B9578EB
-P 10800 7100
-F 0 "U4" H 11000 7000 50  0000 L CNN
-F 1 "NUP2202" H 11000 6900 50  0000 L CNN
-F 2 "Package_TO_SOT_SMD:SOT-363_SC-70-6" H 10880 7175 50  0001 C CNN
-F 3 "http://www.onsemi.ru.com/pub_link/Collateral/NUP2202W1-D.PDF" H 10880 7175 50  0001 C CNN
-F 4 "2533276" H 2250 1750 50  0001 C CNN "Part Number"
-F 5 "Farnell" H 2250 1750 50  0001 C CNN "Supplier"
-	1    10800 7100
+P 10950 7100
+F 0 "U4" H 11150 7000 50  0000 L CNN
+F 1 "NUP2202" H 11150 6900 50  0000 L CNN
+F 2 "Package_TO_SOT_SMD:SOT-363_SC-70-6" H 11030 7175 50  0001 C CNN
+F 3 "http://www.onsemi.ru.com/pub_link/Collateral/NUP2202W1-D.PDF" H 11030 7175 50  0001 C CNN
+F 4 "2533276" H 2400 1750 50  0001 C CNN "Part Number"
+F 5 "Farnell" H 2400 1750 50  0001 C CNN "Supplier"
+	1    10950 7100
 	1    0    0    -1
 $EndComp
@@
 L power:+5V #PWR0114
 U 1 1 5B9579C7
-P 10800 6750
-F 0 "#PWR0114" H 10800 6600 50  0001 C CNN
-F 1 "+5V" H 10815 6923 50  0000 C CNN
-F 2 "" H 10800 6750 50  0001 C CNN
-F 3 "" H 10800 6750 50  0001 C CNN
-	1    10800 6750
-	1    0    0    -1
-$EndComp
-Wire Wire Line
-	10800 6900 10800 6750
+P 10950 6750
+F 0 "#PWR0114" H 10950 6600 50  0001 C CNN
+F 1 "+5V" H 10965 6923 50  0000 C CNN
+F 2 "" H 10950 6750 50  0001 C CNN
+F 3 "" H 10950 6750 50  0001 C CNN
+	1    10950 6750
+	1    0    0    -1
+$EndComp
+Wire Wire Line
+	10950 6900 10950 6750
 $Comp
 L power:GND #PWR0115
 U 1 1 5B958582
-P 10800 7450
-F 0 "#PWR0115" H 10800 7200 50  0001 C CNN
-F 1 "GND" H 10805 7277 50  0000 C CNN
-F 2 "" H 10800 7450 50  0001 C CNN
-F 3 "" H 10800 7450 50  0001 C CNN
-	1    10800 7450
-	1    0    0    -1
-$EndComp
-Wire Wire Line
-	10800 7300 10800 7450
-Wire Wire Line
-	10350 7100 10600 7100
-Wire Wire Line
-	11000 7100 11300 7100
+P 10950 7450
+F 0 "#PWR0115" H 10950 7200 50  0001 C CNN
+F 1 "GND" H 10955 7277 50  0000 C CNN
+F 2 "" H 10950 7450 50  0001 C CNN
+F 3 "" H 10950 7450 50  0001 C CNN
+	1    10950 7450
+	1    0    0    -1
+$EndComp
+Wire Wire Line
+	10950 7300 10950 7450
+Wire Wire Line
+	10500 7100 10750 7100
+Wire Wire Line
+	11150 7100 11450 7100
 $Comp
 L Regulator_Linear:TPS793333-EP U2
@@
 Text Notes 2650 4350 0    50   ~ 0
 Mounting holes, M2.5
-Text Label 10350 7100 0    50   ~ 0
+Text Label 11450 7100 0    50   ~ 0
 USB_P
-Text Label 11100 7100 0    50   ~ 0
+Text Label 10500 7100 0    50   ~ 0
 USB_N
-$Comp
-L DX07P024AJ1R1500:DX07P024AJ1R1500 J2
-U 1 1 5C01B0D3
-P 13100 7050
-F 0 "J2" H 13100 7917 50  0000 C CNN
-F 1 "DX07P024AJ1R1500" H 13100 7826 50  0000 C CNN
-F 2 "lib_fp:DX07P024AJ1R1500" H 13100 7050 50  0001 L BNN
-F 3 "None" H 13100 7050 50  0001 L BNN
-F 4 "DX07P024AJ1R1500" H 13100 7050 50  0001 L BNN "Part Number"
-F 5 "DigiKey" H 13100 7050 50  0001 L BNN "Supplier"
-	1    13100 7050
-	1    0    0    -1
-$EndComp
-Wire Wire Line
-	12600 7150 12150 7150
-Wire Wire Line
-	12600 7250 12150 7250
-$Comp
-L Device:R R4
-U 1 1 5C02A8CD
-P 11850 7250
-F 0 "R4" H 11780 7204 50  0000 R CNN
-F 1 "5k1" H 11780 7295 50  0000 R CNN
-F 2 "Resistor_SMD:R_0805_2012Metric_Pad1.15x1.40mm_HandSolder" V 11780 7250 50  0001 C CNN
-F 3 "~" H 11850 7250 50  0001 C CNN
-	1    11850 7250
-	-1   0    0    1
-$EndComp
-Wire Wire Line
-	11850 7050 12600 7050
-$Comp
-L power:GND #PWR03
-U 1 1 5C02B867
-P 11850 7400
-F 0 "#PWR03" H 11850 7150 50  0001 C CNN
-F 1 "GND" H 11855 7227 50  0000 C CNN
-F 2 "" H 11850 7400 50  0001 C CNN
-F 3 "" H 11850 7400 50  0001 C CNN
-	1    11850 7400
-	1    0    0    -1
-$EndComp
-Wire Wire Line
-	11850 7050 11850 7100
-NoConn ~ 12600 6450
-NoConn ~ 12600 6550
-NoConn ~ 12600 6650
-NoConn ~ 12600 6750
-NoConn ~ 12600 6850
-NoConn ~ 12600 6950
-NoConn ~ 12600 7350
-NoConn ~ 12600 7450
-NoConn ~ 12600 7550
-NoConn ~ 12600 7650
-NoConn ~ 13600 6550
 NoConn ~ 8050 2200
 NoConn ~ 8050 3200
@@
 NoConn ~ 9250 2500
 NoConn ~ 9250 2400
-Wire Wire Line
-	13600 6450 13750 6450
-Wire Wire Line
-	13750 6450 13750 6300
-Wire Wire Line
-	13600 7650 13750 7650
-Wire Wire Line
-	13750 7650 13750 7750
 $Comp
 L Graphic:Logo_Open_Hardware_Small G1
@@
 	0    1    1    0
 $EndComp
+$Comp
+L reversible_micro_usb:reversible_micro_usb J2
+U 1 1 5C79BAD9
+P 13050 6700
+F 0 "J2" H 13050 6775 50  0000 C CNN
+F 1 "reversible_micro_usb" H 13050 6684 50  0000 C CNN
+F 2 "lib_fp:reversible_micro_usb" H 13050 6700 50  0001 C CNN
+F 3 "" H 13050 6700 50  0001 C CNN
+	1    13050 6700
+	1    0    0    -1
+$EndComp
+$Comp
+L power:GND #PWR03
+U 1 1 5C79BD83
+P 12500 7550
+F 0 "#PWR03" H 12500 7300 50  0001 C CNN
+F 1 "GND" H 12505 7377 50  0000 C CNN
+F 2 "" H 12500 7550 50  0001 C CNN
+F 3 "" H 12500 7550 50  0001 C CNN
+	1    12500 7550
+	1    0    0    -1
+$EndComp
+Wire Wire Line
+	12650 7350 12500 7350
+Wire Wire Line
+	12500 7350 12500 7450
+Wire Wire Line
+	12650 7450 12500 7450
+Connection ~ 12500 7450
+Wire Wire Line
+	12500 7450 12500 7550
+$Comp
+L power:GND #PWR05
+U 1 1 5C79E9B0
+P 13600 7550
+F 0 "#PWR05" H 13600 7300 50  0001 C CNN
+F 1 "GND" H 13605 7377 50  0000 C CNN
+F 2 "" H 13600 7550 50  0001 C CNN
+F 3 "" H 13600 7550 50  0001 C CNN
+	1    13600 7550
+	1    0    0    -1
+$EndComp
+Wire Wire Line
+	13450 7450 13600 7450
+Wire Wire Line
+	13600 7450 13600 7550
+Wire Wire Line
+	13450 7350 13600 7350
+Wire Wire Line
+	13600 7350 13600 7450
+Connection ~ 13600 7450
+$Comp
+L power:+5V #PWR04
+U 1 1 5C7A43F8
+P 13600 6750
+F 0 "#PWR04" H 13600 6600 50  0001 C CNN
+F 1 "+5V" H 13615 6923 50  0000 C CNN
+F 2 "" H 13600 6750 50  0001 C CNN
+F 3 "" H 13600 6750 50  0001 C CNN
+	1    13600 6750
+	1    0    0    -1
+$EndComp
+Wire Wire Line
+	13450 6850 13600 6850
+Wire Wire Line
+	13600 6850 13600 6750
+Wire Wire Line
+	13450 6950 13600 6950
+Wire Wire Line
+	13600 6950 13600 6850
+Connection ~ 13600 6850
+Text Label 12450 6850 2    50   ~ 0
+USB_N
+Wire Wire Line
+	12450 6850 12550 6850
+Wire Wire Line
+	12550 6850 12550 6950
+Wire Wire Line
+	12550 6950 12650 6950
+Wire Wire Line
+	12650 6850 12550 6850
+Connection ~ 12550 6850
+Text Label 12450 7100 2    50   ~ 0
+USB_P
+Wire Wire Line
+	12650 7200 12550 7200
+Wire Wire Line
+	12550 7200 12550 7100
+Wire Wire Line
+	12450 7100 12550 7100
+Connection ~ 12550 7100
+Wire Wire Line
+	12550 7100 12650 7100
 $EndSCHEMATC
