File: OpenThermalCamera.sch (KiCad schematic (older format))
At the start: 23 parts, among them J1 Conn_ARM_JTAG_SWD_10, J2 DX07P024AJ1R1500, SW1 PB_Bootloader, U1 MLX90640, U2 TPS793333-EP, U3 STM32F042F6Px, U4 NUP2202

Commit message: Fixed reversible microusb footprint
Parts:
- removed D1: LED_Dual_ACAC, LED_SMD:LED_Cree-PLCC4_2x2mm_CW, symbol Device:LED_Dual_ACAC
- removed J1: Conn_ARM_JTAG_SWD_10, Connector_PinHeader_1.27mm:PinHeader_2x05_P1.27mm_Vertical_SMD, symbol Connector:Conn_ARM_JTAG_SWD_10
- removed U2: TPS793333-EP, Package_TO_SOT_SMD:SOT-23-5_HandSoldering, symbol Regulator_Linear:TPS793333-EP
- added J1: Conn_01x05_Female, Connector_PinHeader_1.27mm:PinHeader_1x05_P1.27mm_Vertical, symbol Connector:Conn_01x05_Female
- added J3: micro5p_reversible_edley_technology, lib_fp:reversible_micro_usb, symbol micro5p_reversible_edley_technology:micro5p_reversible_edley_technology
- added U2: TPS79333-EP, Package_TO_SOT_SMD:SOT-23-5, symbol Regulator_Linear:TPS79333-EP
- C1: mfr# (none) -> VJ0805G225KXYTW1BC
- C2: mfr# (none) -> 885012207011
- C3, C6: mfr# (none) -> 0805B104K250CT
- C4: value 1uF -> 10uF; Part Number 2534058 -> (none); Supplier Farnell -> (none); mfr# (none) -> C2012X5R1C106K085AC
- C5: Part Number 2496943 -> (none); Supplier Farnell -> (none); mfr# (none) -> 0805B104K250CT
- G1: DNP (none) -> 1
- J2: Part Number DX07P024AJ1R1500 -> 656-DX07P024AJ1R1500; Supplier DigiKey -> Mouser; mfr (none) -> JAE Electronics; mfr# (none) -> DX07P024AJ1R1500
- MH1, MH2: DNP (none) -> 1; Part Number / -> (none); Supplier / -> (none)
- R1: value 10k -> 50k; Part Number 2502786 -> (none); Supplier Farnell -> (none); mfr# (none) -> CRCW080551K0JNEA
- R2, R3: Part Number 1653013 -> (none); Supplier Farnell -> (none); mfr# (none) -> CRCW08054K70FKEA
- R4: mfr# (none) -> CRCW08055K10FKEAC
- R5: value 10R -> 1k; mfr# (none) -> CRCW08051K00FKEAC
- R6: value 130R -> 1k; mfr# (none) -> CRCW08051K00FKEAC
- SW1: DNP (none) -> 1; Part Number 2468741 -> /; Supplier Farnell -> /
- U1: Part Number / -> 482-MLX90640ESFBABSP; Supplier / -> Mouser; mfr (none) -> Melexis; mfr# (none) -> MLX90640ESF-BAB-000-SP
- U3: Part Number 2469549 -> 511-STM32F042F6P6TR; Supplier Farnell -> Mouser; mfr (none) -> STMicroelectronics; mfr# (none) -> STM32F042F6P6
- U4: mfr (none) -> ON SEMICONDUCTOR; mfr# (none) -> NUP2202W1T2G
Connections:
- net labels removed: BLUE_LED, RED_LED
- wire segments 58 -> 79
- no-connect marks 22 -> 21
Other:
- note added: "Boot selector and DFU jump possibility"
- note added: "USB TypeC and Micro with ESD protection"
- note removed: "Boot selector"
- note removed: "Indicator Blue/Red LED"
- note removed: "USB connection and ESD protection"
- moved on the sheet: C1, C2, C3, C5, C6, MH1, MH2, R1, R2, R3, R4, SW1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
